File: RibbonCable_MB_BreakdownBoard/RibbonCable_MB_BreakdownBoard.kicad_pcb (KiCad board)
At the start: 2 copper layers, 60 x 35 mm, 18 parts

Commit message: New boards
Parts:
- moved Motor_E 0.30 mm to (127.3, 93.0)
- moved Motor_X 0.30 mm to (127.3, 85.0)
- moved HEAT 0.10 mm to (113.1, 86.4)
Routing:
- net /Heat+: track 18.8 -> 23.0 mm
- net /HEAT_GND: track 20.4 -> 23.3 mm
- net Net-(Motor_X1-Pad4): track 16.9 -> 14.8 mm
- net Net-(Motor_X1-Pad3): track 13.1 -> 11.1 mm
- net Net-(Ribbon1-Pad1): track 14.0 -> 15.3 mm
- net Net-(Motor_E1-Pad1): track 19.3 -> 18.1 mm
- net Net-(Motor_E1-Pad4): track 26.0 -> 27.0 mm
- net Net-(Motor_E1-Pad3): track 21.3 -> 22.2 mm
- net Net-(BLTouch1-Pad1): track 14.5 -> 15.2 mm
- net Net-(Ribbon1-Pad7): track 21.0 -> 21.8 mm
- net Net-(BLTouch1-Pad2): track 15.5 -> 16.1 mm
