File: Transfer_Board/Transfer_Board.kicad_pcb (KiCad board)
At the start: 2 copper layers, 51 x 53 mm, 13 parts

Commit message: New boards
Parts:
- added REF**: OSHW-Logo2_7.3x6mm_SilkScreen, Symbol:OSHW-Logo2_7.3x6mm_SilkScreen, F.Cu at (134.4, 95.8)
Other:
- board text added: "CR-10S Pro Transfer board"
- board text added: "PT"
